File: d.kicad_pcb (KiCad board)
At the start: 2 copper layers, 241 x 191.5 mm, 114 parts, among them J1 Conn_01x18_Pin, J2 Conn_01x03_Pin, K1 Fujitsu_FTR-LYCA005x, K2 Fujitsu_FTR-LYCA005x, K3 Fujitsu_FTR-LYCA005x, K4 Fujitsu_FTR-LYCA005x, K5 Fujitsu_FTR-LYCA005x, K6 Fujitsu_FTR-LYCA005x, K7 Fujitsu_FTR-LYCA005x, K9 Fujitsu_FTR-LYCA005x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

Commit message: Add files via upload
Parts:
- added J3: Conn_01x04_Pin, Connector_PinHeader_2.00mm:PinHeader_1x04_P2.00mm_Vertical, F.Cu at (210.5, 49.0)
- moved U7 25.9 mm to (214.4, 187.4)
- moved BT2 1.80 mm to (218.4, 29.0)
Connections:
- BT2 pad 1: Net-(BT2-+) -> VCC
- BT2 pad 2: Earth -> Net-(BT2--)
