File: smps/smps.kicad_pcb (KiCad board)
At the start: 2 copper layers, 103.5 x 95 mm, 35 parts, among them J1 Conn_01x02_Pin, J2 Conn_01x03_Pin, U1 VIPer22AS, U2 GP2S700HCP, U3 TL431D

Commit message: Add files via upload
Other:
- board size 103.5 x 95 mm -> 103.5 x 99 mm
Changed lines of the file:
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@@
 	(gr_rect
 		(start 74.5 36.5)
-		(end 178 131.5)
+		(end 178 135.5)
 		(stroke
 			(width 0.05)
